File: Adapter Boards/Wi07 Adapter.sch (EAGLE design)
At the start: 3 parts, among them U1 WI07-12FULL

Commit message: Adding new ESP03 Adapter board; Fix minor errors in library
Parts:
- U1: device Wi07:WI07-12FULL -> ESP:WI07-12FULL
Changed lines of the file:
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@@
 </classes>
 <parts>
-<part name="U1" library="Wi07" deviceset="WI07-12" device="FULL"/>
 <part name="JP1" library="SparkFun-Connectors" deviceset="M08" device=""/>
 <part name="JP2" library="SparkFun-Connectors" deviceset="M08" device=""/>
+<part name="U1" library="ESP" deviceset="WI07-12" device="FULL"/>
 </parts>
 <sheets>
@@
 </plain>
 <instances>
-<instance part="U1" gate="G$1" x="73.66" y="15.24"/>
 <instance part="JP1" gate="G$1" x="40.64" y="55.88"/>
 <instance part="JP2" gate="G$1" x="104.14" y="55.88" rot="MR0"/>
+<instance part="U1" gate="G$1" x="73.66" y="55.88"/>
 </instances>
 <busses>
@@
 <segment>
 <pinref part="JP1" gate="G$1" pin="1"/>
+<wire x1="45.72" y1="48.26" x2="53.34" y2="48.26" width="0.1524" layer="91"/>
 <pinref part="U1" gate="G$1" pin="VCC"/>
-<wire x1="45.72" y1="48.26" x2="53.34" y2="48.26" width="0.1524" layer="91"/>
 </segment>
 </net>
@@
 <segment>
 <pinref part="JP1" gate="G$1" pin="2"/>
+<wire x1="45.72" y1="50.8" x2="53.34" y2="50.8" width="0.1524" layer="91"/>
 <pinref part="U1" gate="G$1" pin="13"/>
-<wire x1="45.72" y1="50.8" x2="53.34" y2="50.8" width="0.1524" layer="91"/>
 </segment>
 </net>
 <net name="N$3" class="0">
 <segment>
-<pinref part="U1" gate="G$1" pin="12"/>
 <pinref part="JP1" gate="G$1" pin="3"/>
 <wire x1="53.34" y1="53.34" x2="45.72" y2="53.34" width="0.1524" layer="91"/>
+<pinref part="U1" gate="G$1" pin="12"/>
 </segment>
 </net>
@@
 <segment>
 <pinref part="JP1" gate="G$1" pin="4"/>
+<wire x1="45.72" y1="55.88" x2="53.34" y2="55.88" width="0.1524" layer="91"/>
 <pinref part="U1" gate="G$1" pin="14"/>
-<wire x1="45.72" y1="55.88" x2="53.34" y2="55.88" width="0.1524" layer="91"/>
 </segment>
 </net>
 <net name="N$5" class="0">
 <segment>
-<pinref part="U1" gate="G$1" pin="16"/>
 <pinref part="JP1" gate="G$1" pin="5"/>
 <wire x1="53.34" y1="58.42" x2="45.72" y2="58.42" width="0.1524" layer="91"/>
+<pinref part="U1" gate="G$1" pin="16"/>
 </segment>
 </net>
@@
 <segment>
 <pinref part="JP1" gate="G$1" pin="6"/>
+<wire x1="45.72" y1="60.96" x2="53.34" y2="60.96" width="0.1524" layer="91"/>
 <pinref part="U1" gate="G$1" pin="CH_PD"/>
-<wire x1="45.72" y1="60.96" x2="53.34" y2="60.96" width="0.1524" layer="91"/>
 </segment>
 </net>
 <net name="N$7" class="0">
 <segment>
-<pinref part="U1" gate="G$1" pin="ADC"/>
 <pinref part="JP1" gate="G$1" pin="7"/>
 <wire x1="53.34" y1="63.5" x2="45.72" y2="63.5" width="0.1524" layer="91"/>
+<pinref part="U1" gate="G$1" pin="ADC"/>
 </segment>
 </net>
@@
 <segment>
 <pinref part="JP1" gate="G$1" pin="8"/>
+<wire x1="45.72" y1="66.04" x2="53.34" y2="66.04" width="0.1524" layer="91"/>
 <pinref part="U1" gate="G$1" pin="RESET"/>
-<wire x1="45.72" y1="66.04" x2="53.34" y2="66.04" width="0.1524" layer="91"/>
 </segment>
 </net>
 <net name="N$9" class="0">
 <segment>
-<pinref part="U1" gate="G$1" pin="TXD"/>
 <pinref part="JP2" gate="G$1" pin="8"/>
 <wire x1="93.98" y1="66.04" x2="99.06" y2="66.04" width="0.1524" layer="91"/>
+<pinref part="U1" gate="G$1" pin="TXD"/>
 </segment>
 </net>
@@
 <segment>
 <pinref part="JP2" gate="G$1" pin="7"/>
+<wire x1="99.06" y1="63.5" x2="93.98" y2="63.5" width="0.1524" layer="91"/>
 <pinref part="U1" gate="G$1" pin="RXD"/>
-<wire x1="99.06" y1="63.5" x2="93.98" y2="63.5" width="0.1524" layer="91"/>
 </segment>
 </net>
 <net name="N$11" class="0">
 <segment>
-<pinref part="U1" gate="G$1" pin="4"/>
 <pinref part="JP2" gate="G$1" pin="6"/>
 <wire x1="93.98" y1="60.96" x2="99.06" y2="60.96" width="0.1524" layer="91"/>
+<pinref part="U1" gate="G$1" pin="4"/>
 </segment>
 </net>
@@
 <segment>
 <pinref part="JP2" gate="G$1" pin="5"/>
+<wire x1="99.06" y1="58.42" x2="93.98" y2="58.42" width="0.1524" layer="91"/>
 <pinref part="U1" gate="G$1" pin="5"/>
-<wire x1="99.06" y1="58.42" x2="93.98" y2="58.42" width="0.1524" layer="91"/>
 </segment>
 </net>
 <net name="N$13" class="0">
 <segment>
-<pinref part="U1" gate="G$1" pin="0"/>
 <pinref part="JP2" gate="G$1" pin="4"/>
 <wire x1="93.98" y1="55.88" x2="99.06" y2="55.88" width="0.1524" layer="91"/>
+<pinref part="U1" gate="G$1" pin="0"/>
 </segment>
 </net>
@@
 <segment>
 <pinref part="JP2" gate="G$1" pin="3"/>
+<wire x1="99.06" y1="53.34" x2="93.98" y2="53.34" width="0.1524" layer="91"/>
 <pinref part="U1" gate="G$1" pin="2"/>
-<wire x1="99.06" y1="53.34" x2="93.98" y2="53.34" width="0.1524" layer="91"/>
 </segment>
 </net>
 <net name="N$15" class="0">
 <segment>
-<pinref part="U1" gate="G$1" pin="15"/>
 <pinref part="JP2" gate="G$1" pin="2"/>
 <wire x1="93.98" y1="50.8" x2="99.06" y2="50.8" width="0.1524" layer="91"/>
+<pinref part="U1" gate="G$1" pin="15"/>
 </segment>
 </net>
@@
 <segment>
 <pinref part="JP2" gate="G$1" pin="1"/>
+<wire x1="99.06" y1="48.26" x2="93.98" y2="48.26" width="0.1524" layer="91"/>
 <pinref part="U1" gate="G$1" pin="GND"/>
-<wire x1="99.06" y1="48.26" x2="93.98" y2="48.26" width="0.1524" layer="91"/>
 </segment>
 </net>
