File: Adapter Boards/ESP03 Adapter.sch (EAGLE design)
At the start: 3 parts, among them U1 ESP03

Commit message: Added OSHW logos
Parts:
- added LOGO1: OSHW-LOGOM, SparkFun-Aesthetics:OSHW-LOGOM
- renumbered JP1 to 1, JP2 to 2
Changed lines of the file:
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@@
 <parts>
 <part name="U1" library="ESP" deviceset="ESP03" device=""/>
-<part name="JP1" library="SparkFun-Connectors" deviceset="M07" device=""/>
-<part name="JP2" library="SparkFun-Connectors" deviceset="M07" device=""/>
+<part name="1" library="SparkFun-Connectors" deviceset="M07" device=""/>
+<part name="2" library="SparkFun-Connectors" deviceset="M07" device=""/>
+<part name="LOGO1" library="SparkFun-Aesthetics" deviceset="OSHW-LOGO" device="M"/>
 </parts>
 <sheets>
@@
 <instances>
 <instance part="U1" gate="G$2" x="71.12" y="45.72"/>
-<instance part="JP1" gate="G$1" x="27.94" y="43.18"/>
-<instance part="JP2" gate="G$1" x="111.76" y="43.18" rot="MR0"/>
+<instance part="1" gate="G$1" x="27.94" y="43.18"/>
+<instance part="2" gate="G$1" x="111.76" y="43.18" rot="MR0"/>
+<instance part="LOGO1" gate="G$1" x="63.5" y="17.78"/>
 </instances>
 <busses>
@@
 <pinref part="U1" gate="G$2" pin="VCC"/>
 <wire x1="91.44" y1="53.34" x2="91.44" y2="58.42" width="0.1524" layer="91"/>
-<pinref part="JP1" gate="G$1" pin="7"/>
+<pinref part="1" gate="G$1" pin="7"/>
 <wire x1="91.44" y1="58.42" x2="33.02" y2="58.42" width="0.1524" layer="91"/>
 <wire x1="33.02" y1="58.42" x2="33.02" y2="53.34" width="0.1524" layer="91"/>
@@
 <wire x1="50.8" y1="53.34" x2="35.56" y2="53.34" width="0.1524" layer="91"/>
 <wire x1="35.56" y1="53.34" x2="35.56" y2="50.8" width="0.1524" layer="91"/>
-<pinref part="JP1" gate="G$1" pin="6"/>
+<pinref part="1" gate="G$1" pin="6"/>
 <wire x1="35.56" y1="50.8" x2="33.02" y2="50.8" width="0.1524" layer="91"/>
 </segment>
@@
 <wire x1="50.8" y1="50.8" x2="38.1" y2="50.8" width="0.1524" layer="91"/>
 <wire x1="38.1" y1="50.8" x2="38.1" y2="48.26" width="0.1524" layer="91"/>
-<pinref part="JP1" gate="G$1" pin="5"/>
+<pinref part="1" gate="G$1" pin="5"/>
 <wire x1="38.1" y1="48.26" x2="33.02" y2="48.26" width="0.1524" layer="91"/>
 </segment>
@@
 <wire x1="50.8" y1="48.26" x2="40.64" y2="48.26" width="0.1524" layer="91"/>
 <wire x1="40.64" y1="48.26" x2="40.64" y2="45.72" width="0.1524" layer="91"/>
-<pinref part="JP1" gate="G$1" pin="4"/>
+<pinref part="1" gate="G$1" pin="4"/>
 <wire x1="40.64" y1="45.72" x2="33.02" y2="45.72" width="0.1524" layer="91"/>
 </segment>
@@
 <wire x1="50.8" y1="45.72" x2="43.18" y2="45.72" width="0.1524" layer="91"/>
 <wire x1="43.18" y1="45.72" x2="43.18" y2="43.18" width="0.1524" layer="91"/>
-<pinref part="JP1" gate="G$1" pin="3"/>
+<pinref part="1" gate="G$1" pin="3"/>
 <wire x1="43.18" y1="43.18" x2="33.02" y2="43.18" width="0.1524" layer="91"/>
 </segment>
@@
 <wire x1="50.8" y1="43.18" x2="45.72" y2="43.18" width="0.1524" layer="91"/>
 <wire x1="45.72" y1="43.18" x2="45.72" y2="40.64" width="0.1524" layer="91"/>
-<pinref part="JP1" gate="G$1" pin="2"/>
+<pinref part="1" gate="G$1" pin="2"/>
 <wire x1="45.72" y1="40.64" x2="33.02" y2="40.64" width="0.1524" layer="91"/>
 </segment>
@@
 <wire x1="50.8" y1="40.64" x2="48.26" y2="40.64" width="0.1524" layer="91"/>
 <wire x1="48.26" y1="40.64" x2="48.26" y2="38.1" width="0.1524" layer="91"/>
-<pinref part="JP1" gate="G$1" pin="1"/>
+<pinref part="1" gate="G$1" pin="1"/>
 <wire x1="48.26" y1="38.1" x2="33.02" y2="38.1" width="0.1524" layer="91"/>
 </segment>
@@
 <wire x1="91.44" y1="50.8" x2="93.98" y2="50.8" width="0.1524" layer="91"/>
 <wire x1="93.98" y1="50.8" x2="93.98" y2="53.34" width="0.1524" layer="91"/>
-<pinref part="JP2" gate="G$1" pin="7"/>
+<pinref part="2" gate="G$1" pin="7"/>
 <wire x1="93.98" y1="53.34" x2="106.68" y2="53.34" width="0.1524" layer="91"/>
 </segment>
@@
 <wire x1="91.44" y1="48.26" x2="96.52" y2="48.26" width="0.1524" layer="91"/>
 <wire x1="96.52" y1="48.26" x2="96.52" y2="50.8" width="0.1524" layer="91"/>
-<pinref part="JP2" gate="G$1" pin="6"/>
+<pinref part="2" gate="G$1" pin="6"/>
 <wire x1="96.52" y1="50.8" x2="106.68" y2="50.8" width="0.1524" layer="91"/>
 </segment>
@@
 <wire x1="93.98" y1="45.72" x2="99.06" y2="45.72" width="0.1524" layer="91"/>
 <wire x1="99.06" y1="45.72" x2="99.06" y2="48.26" width="0.1524" layer="91"/>
-<pinref part="JP2" gate="G$1" pin="5"/>
+<pinref part="2" gate="G$1" pin="5"/>
 <wire x1="99.06" y1="48.26" x2="106.68" y2="48.26" width="0.1524" layer="91"/>
 </segment>
@@
 <wire x1="91.44" y1="43.18" x2="101.6" y2="43.18" width="0.1524" layer="91"/>
 <wire x1="101.6" y1="43.18" x2="101.6" y2="45.72" width="0.1524" layer="91"/>
-<pinref part="JP2" gate="G$1" pin="4"/>
+<pinref part="2" gate="G$1" pin="4"/>
 <wire x1="101.6" y1="45.72" x2="106.68" y2="45.72" width="0.1524" layer="91"/>
 </segment>
@@
 <wire x1="91.44" y1="40.64" x2="104.14" y2="40.64" width="0.1524" layer="91"/>
 <wire x1="104.14" y1="40.64" x2="104.14" y2="43.18" width="0.1524" layer="91"/>
-<pinref part="JP2" gate="G$1" pin="3"/>
+<pinref part="2" gate="G$1" pin="3"/>
 <wire x1="104.14" y1="43.18" x2="106.68" y2="43.18" width="0.1524" layer="91"/>
 </segment>
@@
 <segment>
 <pinref part="U1" gate="G$2" pin="GND"/>
-<pinref part="JP2" gate="G$1" pin="1"/>
+<pinref part="2" gate="G$1" pin="1"/>
 <wire x1="91.44" y1="38.1" x2="106.68" y2="38.1" width="0.1524" layer="91"/>
 </segment>
